Commit message: Adds working packages for the 2 finger models using USB & ros control

File: robotiq_2f_model/model/robotiq_2f_85.urdf.xacro (robot description, xacro)
@@ -3,5 +3,6 @@
 	Coordinate system convention for grippers:
 	The pin of the gripper is along the y-axis, and z-axis points up.
-	The resulting x-axis is considered the palm face, so +y is right, and -y is left.
+	The resulting x-axis is considered the palm face, so +y is right, and -y is left for
+	a right-hand gripper, whatever that means in this gripper.
 	Coarse and precise models:
 	Two granularities for collision are provided, a coarse (default) for quick motion
@@ -12,5 +13,5 @@
 	and update of real hw, and an implementation of the 5-bar transmission with
 	spring transmission for grasp simulation.
-	For grasp simulation, the file c85.gazebo.xacro sets additional parameters such as
+	For grasp simulation, the file 2f85.gazebo.xacro sets additional parameters such as
 	material properties, and simulation parameters.
 -->
@@ -20,8 +21,8 @@
 </xacro:macro -->
 <robot xmlns:xacro="http://ros.org/wiki/xacro">
-	<xacro:macro name="robotiq_c_85" params="parent name precise_collision:=false adaptive_transmission:=false *origin">
+	<xacro:macro name="robotiq_2f_85" params="parent name precise_collision:=false adaptive_transmission:=false *origin">
 		<!-- base -->
 		<joint name="${parent}_${name}_base_joint" type="fixed">
-			<insert_block name="origin"/>
+			<xacro:insert_block name="origin"/>
 			<parent link="${parent}"/>
 			<child link="${name}_base"/>
@@ -35,5 +36,5 @@
 			<visual>
 				<geometry>
-					<mesh filename="package://robotiq_2f_model/model/meshes/c85/visual/base.dae" scale="0.001 0.001 0.001"/>
+					<mesh filename="package://robotiq_2f_model/model/meshes/2f85/visual/base.dae" scale="0.001 0.001 0.001"/>
 				</geometry>
 			</visual>
@@ -55,5 +56,5 @@
 			<collision>
 				<geometry>
-					<mesh filename="package://robotiq_2f_model/model/meshes/c85/collision/base.stl" scale="0.001 0.001 0.001"/>
+					<mesh filename="package://robotiq_2f_model/model/meshes/2f85/collision/base.stl" scale="0.001 0.001 0.001"/>
 				</geometry>
 			</collision>
@@ -66,5 +67,5 @@
 			<child link="${name}_right_driver"/>
 			<axis xyz="1 0 0"/>
-			<limit lower="${0 * 3.141592 / 180}" upper="${41 * 3.141592 / 180}" effort="176" velocity="${110 * 3.141592 / 180}" />
+			<limit lower="${0 * 3.141592 / 180}" upper="${50 * 3.141592 / 180}" effort="60" velocity="${110 * 3.141592 / 180}" />
 		</joint>
 		<link name="${name}_right_driver">
@@ -76,5 +77,5 @@
 			<visual>
 				<geometry>
-					<mesh filename="package://robotiq_2f_model/model/meshes/c85/visual/driver.dae" scale="0.001 0.001 0.001"/>
+					<mesh filename="package://robotiq_2f_model/model/meshes/2f85/visual/driver.dae" scale="0.001 0.001 0.001"/>
 				</geometry>
 			</visual>
@@ -90,5 +91,5 @@
 			<collision>
 				<geometry>
-					<mesh filename="package://robotiq_2f_model/model/meshes/c85/collision/driver.stl" scale="0.001 0.001 0.001"/>
+					<mesh filename="package://robotiq_2f_model/model/meshes/2f85/collision/driver.stl" scale="0.001 0.001 0.001"/>
 				</geometry>
 			</collision>
@@ -119,5 +120,5 @@
 			<visual>
 				<geometry>
-					<mesh filename="package://robotiq_2f_model/model/meshes/c85/visual/coupler.dae" scale="0.001 0.001 0.001"/>
+					<mesh filename="package://robotiq_2f_model/model/meshes/2f85/visual/coupler.dae" scale="0.001 0.001 0.001"/>
 				</geometry>
 			</visual>
@@ -133,5 +134,5 @@
 				<collision>
 					<geometry>
-						<mesh filename="package://robotiq_2f_model/model/meshes/c85/collision/coupler.stl" scale="0.001 0.001 0.001"/>
+						<mesh filename="package://robotiq_2f_model/model/meshes/2f85/collision/coupler.stl" scale="0.001 0.001 0.001"/>
 					</geometry>
 				</collision>
@@ -156,5 +157,5 @@
 			<visual>
 				<geometry>
-					<mesh filename="package://robotiq_2f_model/model/meshes/c85/visual/follower.dae" scale="0.001 0.001 0.001"/>
+					<mesh filename="package://robotiq_2f_model/model/meshes/2f85/visual/follower.dae" scale="0.001 0.001 0.001"/>
 				</geometry>
 			</visual>
@@ -170,5 +171,5 @@
 			<collision>
 				<geometry>
-					<mesh filename="package://robotiq_2f_model/model/meshes/c85/collision/follower.stl" scale="0.001 0.001 0.001"/>
+					<mesh filename="package://robotiq_2f_model/model/meshes/2f85/collision/follower.stl" scale="0.001 0.001 0.001"/>
 				</geometry>
 			</collision>
@@ -187,5 +188,5 @@
 			<visual>
 				<geometry>
-					<mesh filename="package://robotiq_2f_model/model/meshes/c85/visual/pad.dae" scale="0.001 0.001 0.001"/>
+					<mesh filename="package://robotiq_2f_model/model/meshes/2f85/visual/pad.dae" scale="0.001 0.001 0.001"/>
 				</geometry>
 			</visual>
@@ -201,5 +202,5 @@
 			<collision>
 				<geometry>
-					<mesh filename="package://robotiq_2f_model/model/meshes/c85/collision/pad.stl" scale="0.001 0.001 0.001"/>
+					<mesh filename="package://robotiq_2f_model/model/meshes/2f85/collision/pad.stl" scale="0.001 0.001 0.001"/>
 				</geometry>
 			</collision>
@@ -224,5 +225,5 @@
 			<visual>
 				<geometry>
-					<mesh filename="package://robotiq_2f_model/model/meshes/c85/visual/spring_link.dae" scale="0.001 0.001 0.001"/>
+					<mesh filename="package://robotiq_2f_model/model/meshes/2f85/visual/spring_link.dae" scale="0.001 0.001 0.001"/>
 				</geometry>
 			</visual>
@@ -238,5 +239,5 @@
 			<collision>
 				<geometry>
-					<mesh filename="package://robotiq_2f_model/model/meshes/c85/collision/spring_link.stl" scale="0.001 0.001 0.001"/>
+					<mesh filename="package://robotiq_2f_model/model/meshes/2f85/collision/spring_link.stl" scale="0.001 0.001 0.001"/>
 				</geometry>
 			</collision>
@@ -262,5 +263,5 @@
 			<visual>
 				<geometry>
-					<mesh filename="package://robotiq_2f_model/model/meshes/c85/visual/driver.dae" scale="0.001 0.001 0.001"/>
+					<mesh filename="package://robotiq_2f_model/model/meshes/2f85/visual/driver.dae" scale="0.001 0.001 0.001"/>
 				</geometry>
 			</visual>
@@ -276,5 +277,5 @@
 			<collision>
 				<geometry>
-					<mesh filename="package://robotiq_2f_model/model/meshes/c85/collision/driver.stl" scale="0.001 0.001 0.001"/>
+					<mesh filename="package://robotiq_2f_model/model/meshes/2f85/collision/driver.stl" scale="0.001 0.001 0.001"/>
 				</geometry>
 			</collision>
@@ -305,5 +306,5 @@
 			<visual>
 				<geometry>
-					<mesh filename="package://robotiq_2f_model/model/meshes/c85/visual/coupler.dae" scale="0.001 0.001 0.001"/>
+					<mesh filename="package://robotiq_2f_model/model/meshes/2f85/visual/coupler.dae" scale="0.001 0.001 0.001"/>
 				</geometry>
 			</visual>
@@ -319,5 +320,5 @@
 				<collision>
 					<geometry>
-						<mesh filename="package://robotiq_2f_model/model/meshes/c85/collision/coupler.stl" scale="0.001 0.001 0.001"/>
+						<mesh filename="package://robotiq_2f_model/model/meshes/2f85/collision/coupler.stl" scale="0.001 0.001 0.001"/>
 					</geometry>
 				</collision>
@@ -342,5 +343,5 @@
 			<visual>
 				<geometry>
-					<mesh filename="package://robotiq_2f_model/model/meshes/c85/visual/follower.dae" scale="0.001 0.001 0.001"/>
+					<mesh filename="package://robotiq_2f_model/model/meshes/2f85/visual/follower.dae" scale="0.001 0.001 0.001"/>
 				</geometry>
 			</visual>
@@ -356,5 +357,5 @@
 			<collision>
 				<geometry>
-					<mesh filename="package://robotiq_2f_model/model/meshes/c85/collision/follower.stl" scale="0.001 0.001 0.001"/>
+					<mesh filename="package://robotiq_2f_model/model/meshes/2f85/collision/follower.stl" scale="0.001 0.001 0.001"/>
 				</geometry>
 			</collision>
@@ -373,5 +374,5 @@
 			<visual>
 				<geometry>
-					<mesh filename="package://robotiq_2f_model/model/meshes/c85/visual/pad.dae" scale="0.001 0.001 0.001"/>
+					<mesh filename="package://robotiq_2f_model/model/meshes/2f85/visual/pad.dae" scale="0.001 0.001 0.001"/>
 				</geometry>
 			</visual>
@@ -387,5 +388,5 @@
 			<collision>
 				<geometry>
-					<mesh filename="package://robotiq_2f_model/model/meshes/c85/collision/pad.stl" scale="0.001 0.001 0.001"/>
+					<mesh filename="package://robotiq_2f_model/model/meshes/2f85/collision/pad.stl" scale="0.001 0.001 0.001"/>
 				</geometry>
 			</collision>
@@ -410,5 +411,5 @@
 			<visual>
 				<geometry>
-					<mesh filename="package://robotiq_2f_model/model/meshes/c85/visual/spring_link.dae" scale="0.001 0.001 0.001"/>
+					<mesh filename="package://robotiq_2f_model/model/meshes/2f85/visual/spring_link.dae" scale="0.001 0.001 0.001"/>
 				</geometry>
 			</visual>
@@ -424,9 +425,18 @@
 			<collision>
 				<geometry>
-					<mesh filename="package://robotiq_2f_model/model/meshes/c85/collision/spring_link.stl" scale="0.001 0.001 0.001"/>
-				</geometry>
-			</collision>
-			</xacro:if>
-		</link>
+					<mesh filename="package://robotiq_2f_model/model/meshes/2f85/collision/spring_link.stl" scale="0.001 0.001 0.001"/>
+				</geometry>
+			</collision>
+			</xacro:if>
+		</link>
+		<transmission name="${name}_right_driver_trans">
+			<type>transmission_interface/SimpleTransmission</type>
+			<joint name="${name}_right_driver_joint">
+				<hardwareInterface>PositionJointInterface</hardwareInterface>
+			</joint>
+			<actuator name="${name}_right_driver_motor">
+				<mechanicalReduction>1</mechanicalReduction>
+			</actuator>
+		</transmission>
 	</xacro:macro>
 </robot>

Commit message: Adds a parameter to add Pads or not to the URDF gripper

File: robotiq_2f_model/model/robotiq_2f_85.urdf.xacro (robot description, xacro)
@@ -21,5 +21,5 @@
 </xacro:macro -->
 <robot xmlns:xacro="http://ros.org/wiki/xacro">
-	<xacro:macro name="robotiq_2f_85" params="parent name precise_collision:=false adaptive_transmission:=false *origin">
+	<xacro:macro name="robotiq_2f_85" params="parent name precise_collision:=false adaptive_transmission:=false with_pads=true *origin">
 		<!-- base -->
 		<joint name="${parent}_${name}_base_joint" type="fixed">
@@ -150,9 +150,4 @@
 		</joint>
 		<link name="${name}_right_follower">
-			<!-- inertial>
-				<mass value="0.1"/>
-				<origin xyz="0 0 0.055"  />
-				<cylinder_inertia radius="0.06" length="0.11" mass="0.1"/>
-			</inertial -->
 			<visual>
 				<geometry>
@@ -176,35 +171,33 @@
 			</xacro:if>
 		</link>
-		<joint name="${name}_right_pad_joint" type="fixed">
-			<parent link="${name}_right_follower"/>
-			<child link="${name}_right_pad"/>
-		</joint>
-		<link name="${name}_right_pad">
-			<!-- inertial>
-				<mass value="0.1"/>
-				<origin xyz="0 0 0.055"  />
-				<cylinder_inertia radius="0.06" length="0.11" mass="0.1"/>
-			</inertial -->
-			<visual>
-				<geometry>
-					<mesh filename="package://robotiq_2f_model/model/meshes/2f85/visual/pad.dae" scale="0.001 0.001 0.001"/>
-				</geometry>
-			</visual>
-			<xacro:unless value="${precise_collision}">
-			<collision>
-				<origin xyz="0 -0.02 0.03" rpy="0 0 0"/>
-				<geometry>
-					<box size="0.04 0.02 0.06"/>
-				</geometry>
-			</collision>
-			</xacro:unless>
-			<xacro:if value="${precise_collision}">
-			<collision>
-				<geometry>
-					<mesh filename="package://robotiq_2f_model/model/meshes/2f85/collision/pad.stl" scale="0.001 0.001 0.001"/>
-				</geometry>
-			</collision>
-			</xacro:if>
-		</link>
+			<joint name="${name}_right_pad_joint" type="fixed">
+				<parent link="${name}_right_follower"/>
+				<child link="${name}_right_pad"/>
+			</joint>
+			<link name="${name}_right_pad">
+				<!-- If no pad, it just leave the visual and the collision empty such that the hw structure remains, e.g. for moveit! -->
+				<xacro:if value="${with_pads}">
+					<visual>
+						<geometry>
+							<mesh filename="package://robotiq_2f_model/model/meshes/2f85/visual/pad.dae" scale="0.001 0.001 0.001"/>
+						</geometry>
+					</visual>
+					<xacro:unless value="${precise_collision}">
+					<collision>
+						<origin xyz="0 -0.02 0.03" rpy="0 0 0"/>
+						<geometry>
+							<box size="0.04 0.02 0.06"/>
+						</geometry>
+					</collision>
+					</xacro:unless>
+					<xacro:if value="${precise_collision}">
+					<collision>
+						<geometry>
+							<mesh filename="package://robotiq_2f_model/model/meshes/2f85/collision/pad.stl" scale="0.001 0.001 0.001"/>
+						</geometry>
+					</collision>
+					</xacro:if>
+				</xacro:if>
+			</link>
 		<joint name="${name}_right_spring_link_joint" type="revolute">
 			<origin xyz="0 0.012 0.0614" rpy="0 0 0"/>
@@ -336,9 +329,4 @@
 		</joint>
 		<link name="${name}_left_follower">
-			<!-- inertial>
-				<mass value="0.1"/>
-				<origin xyz="0 0 0.055"  />
-				<cylinder_inertia radius="0.06" length="0.11" mass="0.1"/>
-			</inertial -->
 			<visual>
 				<geometry>
@@ -367,28 +355,26 @@
 		</joint>
 		<link name="${name}_left_pad">
-			<!-- inertial>
-				<mass value="0.1"/>
-				<origin xyz="0 0 0.055"  />
-				<cylinder_inertia radius="0.06" length="0.11" mass="0.1"/>
-			</inertial -->
-			<visual>
-				<geometry>
-					<mesh filename="package://robotiq_2f_model/model/meshes/2f85/visual/pad.dae" scale="0.001 0.001 0.001"/>
-				</geometry>
-			</visual>
-			<xacro:unless value="${precise_collision}">
-			<collision>
-				<origin xyz="0 -0.02 0.03" rpy="0 0 0"/>
-				<geometry>
-					<box size="0.04 0.02 0.06"/>
-				</geometry>
-			</collision>
-			</xacro:unless>
-			<xacro:if value="${precise_collision}">
-			<collision>
-				<geometry>
-					<mesh filename="package://robotiq_2f_model/model/meshes/2f85/collision/pad.stl" scale="0.001 0.001 0.001"/>
-				</geometry>
-			</collision>
+			<!-- If no pad, it just leave the visual and the collision empty such that the hw structure remains, e.g. for moveit! -->
+			<xacro:if value="${with_pads}">
+				<visual>
+					<geometry>
+						<mesh filename="package://robotiq_2f_model/model/meshes/2f85/visual/pad.dae" scale="0.001 0.001 0.001"/>
+					</geometry>
+				</visual>
+				<xacro:unless value="${precise_collision}">
+				<collision>
+					<origin xyz="0 -0.02 0.03" rpy="0 0 0"/>
+					<geometry>
+						<box size="0.04 0.02 0.06"/>
+					</geometry>
+				</collision>
+				</xacro:unless>
+				<xacro:if value="${precise_collision}">
+				<collision>
+					<geometry>
+						<mesh filename="package://robotiq_2f_model/model/meshes/2f85/collision/pad.stl" scale="0.001 0.001 0.001"/>
+					</geometry>
+				</collision>
+				</xacro:if>
 			</xacro:if>
 		</link>

Commit message: Adjust more precisely the non-precise collision geometry

File: robotiq_2f_model/model/robotiq_2f_85.urdf.xacro (robot description, xacro)
@@ -84,5 +84,5 @@
 				<origin xyz="0 0.02 0" rpy="-0.1 0 0"/>
 				<geometry>
-					<box size="0.04 0.04 0.02"/>
+					<box size="0.02 0.04 0.02"/>
 				</geometry>
 			</collision>
@@ -127,5 +127,5 @@
 				<origin xyz="0 0.0 0.025" rpy="-1.7 0 0"/>
 				<geometry>
-					<box size="0.04 0.065 0.02"/>
+					<box size="0.03 0.065 0.02"/>
 				</geometry>
 			</collision>
@@ -157,7 +157,7 @@
 			<xacro:unless value="${precise_collision}">
 			<collision>
-				<origin xyz="0 -0.02 0.03" rpy="0 0 0"/>
-				<geometry>
-					<box size="0.04 0.02 0.06"/>
+				<origin xyz="0 -0.018 0.022" rpy="0 0 0"/>
+				<geometry>
+					<box size="0.02 0.015 0.048"/>
 				</geometry>
 			</collision>
@@ -171,33 +171,35 @@
 			</xacro:if>
 		</link>
-			<joint name="${name}_right_pad_joint" type="fixed">
-				<parent link="${name}_right_follower"/>
-				<child link="${name}_right_pad"/>
-			</joint>
-			<link name="${name}_right_pad">
-				<!-- If no pad, it just leave the visual and the collision empty such that the hw structure remains, e.g. for moveit! -->
-				<xacro:if value="${with_pads}">
-					<visual>
-						<geometry>
-							<mesh filename="package://robotiq_2f_model/model/meshes/2f85/visual/pad.dae" scale="0.001 0.001 0.001"/>
-						</geometry>
-					</visual>
-					<xacro:unless value="${precise_collision}">
-					<collision>
-						<origin xyz="0 -0.02 0.03" rpy="0 0 0"/>
-						<geometry>
-							<box size="0.04 0.02 0.06"/>
-						</geometry>
-					</collision>
-					</xacro:unless>
-					<xacro:if value="${precise_collision}">
-					<collision>
-						<geometry>
-							<mesh filename="package://robotiq_2f_model/model/meshes/2f85/collision/pad.stl" scale="0.001 0.001 0.001"/>
-						</geometry>
-					</collision>
-					</xacro:if>
-				</xacro:if>
-			</link>
+		<joint name="${name}_right_pad_joint" type="fixed">
+			<parent link="${name}_right_follower"/>
+			<child link="${name}_right_pad"/>
+		</joint>
+		<link name="${name}_right_pad">
+			<!-- inertial>
+				<mass value="0.1"/>
+				<origin xyz="0 0 0.055"  />
+				<cylinder_inertia radius="0.06" length="0.11" mass="0.1"/>
+			</inertial -->
+			<visual>
+				<geometry>
+					<mesh filename="package://robotiq_2f_model/model/meshes/2f85/visual/pad.dae" scale="0.001 0.001 0.001"/>
+				</geometry>
+			</visual>
+			<xacro:unless value="${precise_collision}">
+			<collision>
+				<origin xyz="0 -0.022 0.031" rpy="0 0 0"/>
+				<geometry>
+					<box size="0.02 0.008 0.036"/>
+				</geometry>
+			</collision>
+			</xacro:unless>
+			<xacro:if value="${precise_collision}">
+			<collision>
+				<geometry>
+					<mesh filename="package://robotiq_2f_model/model/meshes/2f85/collision/pad.stl" scale="0.001 0.001 0.001"/>
+				</geometry>
+			</collision>
+			</xacro:if>
+		</link>
 		<joint name="${name}_right_spring_link_joint" type="revolute">
 			<origin xyz="0 0.012 0.0614" rpy="0 0 0"/>
@@ -263,5 +265,5 @@
 				<origin xyz="0 0.02 0" rpy="-0.1 0 0"/>
 				<geometry>
-					<box size="0.04 0.04 0.02"/>
+					<box size="0.02 0.04 0.02"/>
 				</geometry>
 			</collision>
@@ -306,5 +308,5 @@
 				<origin xyz="0 0.0 0.025" rpy="-1.7 0 0"/>
 				<geometry>
-					<box size="0.04 0.065 0.02"/>
+					<box size="0.03 0.065 0.02"/>
 				</geometry>
 			</collision>
@@ -336,7 +338,7 @@
 			<xacro:unless value="${precise_collision}">
 			<collision>
-				<origin xyz="0 -0.02 0.03" rpy="0 0 0"/>
-				<geometry>
-					<box size="0.04 0.02 0.06"/>
+				<origin xyz="0 -0.018 0.022" rpy="0 0 0"/>
+				<geometry>
+					<box size="0.02 0.015 0.048"/>
 				</geometry>
 			</collision>
@@ -355,26 +357,28 @@
 		</joint>
 		<link name="${name}_left_pad">
-			<!-- If no pad, it just leave the visual and the collision empty such that the hw structure remains, e.g. for moveit! -->
-			<xacro:if value="${with_pads}">
-				<visual>
-					<geometry>
-						<mesh filename="package://robotiq_2f_model/model/meshes/2f85/visual/pad.dae" scale="0.001 0.001 0.001"/>
-					</geometry>
-				</visual>
-				<xacro:unless value="${precise_collision}">
-				<collision>
-					<origin xyz="0 -0.02 0.03" rpy="0 0 0"/>
-					<geometry>
-						<box size="0.04 0.02 0.06"/>
-					</geometry>
-				</collision>
-				</xacro:unless>
-				<xacro:if value="${precise_collision}">
-				<collision>
-					<geometry>
-						<mesh filename="package://robotiq_2f_model/model/meshes/2f85/collision/pad.stl" scale="0.001 0.001 0.001"/>
-					</geometry>
-				</collision>
-				</xacro:if>
+			<!-- inertial>
+				<mass value="0.1"/>
+				<origin xyz="0 0 0.055"  />
+				<cylinder_inertia radius="0.06" length="0.11" mass="0.1"/>
+			</inertial -->
+			<visual>
+				<geometry>
+					<mesh filename="package://robotiq_2f_model/model/meshes/2f85/visual/pad.dae" scale="0.001 0.001 0.001"/>
+				</geometry>
+			</visual>
+			<xacro:unless value="${precise_collision}">
+			<collision>
+				<origin xyz="0 -0.022 0.031" rpy="0 0 0"/>
+				<geometry>
+					<box size="0.02 0.008 0.036"/>
+				</geometry>
+			</collision>
+			</xacro:unless>
+			<xacro:if value="${precise_collision}">
+			<collision>
+				<geometry>
+					<mesh filename="package://robotiq_2f_model/model/meshes/2f85/collision/pad.stl" scale="0.001 0.001 0.001"/>
+				</geometry>
+			</collision>
 			</xacro:if>
 		</link>

Commit message: Update robotiq_2f_85.urdf.xacro

File: robotiq_2f_model/model/robotiq_2f_85.urdf.xacro (robot description, xacro)
@@ -21,5 +21,5 @@
 </xacro:macro -->
 <robot xmlns:xacro="http://ros.org/wiki/xacro">
-	<xacro:macro name="robotiq_2f_85" params="parent name precise_collision:=false adaptive_transmission:=false with_pads=true *origin">
+	<xacro:macro name="robotiq_2f_85" params="parent name precise_collision:=false adaptive_transmission:=false with_pads:=true *origin">
 		<!-- base -->
 		<joint name="${parent}_${name}_base_joint" type="fixed">
