Commit message: Update robotiq_2f_85.urdf.xacro
added mimicJoints for gazebo

File: robotiq_2f_model/model/robotiq_2f_85.urdf.xacro (robot description, xacro)
@@ -17,8 +17,13 @@
 -->
 <!-- length is along the z-axis! -->
-<!-- xacro:macro name="cylinder_inertia" params="radius length mass">
-	<inertia ixx="${mass * (3 * radius * radius + length * length) / 12}" iyy="${mass * radius* radius / 2}" izz="${mass * (3 * radius * radius + length * length) / 12}" ixy="0" iyz="0" ixz="0"/>
-</xacro:macro -->
 <robot xmlns:xacro="http://ros.org/wiki/xacro">
+	<xacro:macro name="cylinder_inertia" params="radius length mass">
+		<inertia ixx="${mass * (3 * radius * radius + length * length) / 12}"
+			 iyy="${mass * radius* radius / 2}"
+			 izz="${mass * (3 * radius * radius + length * length) / 12}"
+			 ixy="0"
+			 iyz="0"
+			 ixz="0"/>
+	</xacro:macro>
 	<xacro:macro name="robotiq_2f_85" params="parent name precise_collision:=false adaptive_transmission:=false with_pads:=true *origin">
 		<!-- base -->
@@ -34,4 +39,9 @@
 				<cylinder_inertia radius="0.06" length="0.11" mass="0.1"/>
 			</inertial -->
+			<inertial>
+				<mass value="0.1"/>
+				<origin xyz="0 0 0.055"/>
+				<cylinder_inertia radius="0.06" length="0.11" mass="0.1"/>
+			</inertial>
 			<visual>
 				<geometry>
@@ -75,4 +85,9 @@
 				<cylinder_inertia radius="0.06" length="0.11" mass="0.1"/>
 			</inertial -->
+			<inertial>
+				<mass value="0.1"/>
+				<origin xyz="0 0 0.055"  />
+				<cylinder_inertia radius="0.06" length="0.11" mass="0.1"/>
+			</inertial>
 			<visual>
 				<geometry>
@@ -118,4 +133,9 @@
 				<cylinder_inertia radius="0.06" length="0.11" mass="0.1"/>
 			</inertial -->
+			<inertial>
+				<mass value="0.1"/>
+				<origin xyz="0 0 0.055"  />
+				<cylinder_inertia radius="0.06" length="0.11" mass="0.1"/>
+			</inertial>
 			<visual>
 				<geometry>
@@ -181,4 +201,9 @@
 				<cylinder_inertia radius="0.06" length="0.11" mass="0.1"/>
 			</inertial -->
+			<inertial>
+				<mass value="0.1"/>
+				<origin xyz="0 0 0.055"  />
+				<cylinder_inertia radius="0.06" length="0.11" mass="0.1"/>
+			</inertial>
 			<visual>
 				<geometry>
@@ -218,4 +243,9 @@
 				<cylinder_inertia radius="0.06" length="0.11" mass="0.1"/>
 			</inertial -->
+			<inertial>
+				<mass value="0.1"/>
+				<origin xyz="0 0 0.055"  />
+				<cylinder_inertia radius="0.06" length="0.11" mass="0.1"/>
+			</inertial>
 			<visual>
 				<geometry>
@@ -256,4 +286,9 @@
 				<cylinder_inertia radius="0.06" length="0.11" mass="0.1"/>
 			</inertial -->
+			<inertial>
+				<mass value="0.1"/>
+				<origin xyz="0 0 0.055"  />
+				<cylinder_inertia radius="0.06" length="0.11" mass="0.1"/>
+			</inertial>
 			<visual>
 				<geometry>
@@ -299,4 +334,9 @@
 				<cylinder_inertia radius="0.06" length="0.11" mass="0.1"/>
 			</inertial -->
+			<inertial>
+				<mass value="0.1"/>
+				<origin xyz="0 0 0.055"  />
+				<cylinder_inertia radius="0.06" length="0.11" mass="0.1"/>
+			</inertial>
 			<visual>
 				<geometry>
@@ -362,4 +402,9 @@
 				<cylinder_inertia radius="0.06" length="0.11" mass="0.1"/>
 			</inertial -->
+			<inertial>
+				<mass value="0.1"/>
+				<origin xyz="0 0 0.055"  />
+				<cylinder_inertia radius="0.06" length="0.11" mass="0.1"/>
+			</inertial>
 			<visual>
 				<geometry>
@@ -399,4 +444,9 @@
 				<cylinder_inertia radius="0.06" length="0.11" mass="0.1"/>
 			</inertial -->
+			<inertial>
+				<mass value="0.1"/>
+				<origin xyz="0 0 0.055"  />
+				<cylinder_inertia radius="0.06" length="0.11" mass="0.1"/>
+			</inertial>
 			<visual>
 				<geometry>
@@ -427,6 +477,40 @@
 			<actuator name="${name}_right_driver_motor">
 				<mechanicalReduction>1</mechanicalReduction>
+				<hardwareInterface>PositionJointInterface</hardwareInterface>
 			</actuator>
 		</transmission>
+		<gazebo>
+		        <!-- loading plugin: mimic joints works in gazebo now -->
+		    <plugin filename="libroboticsgroup_gazebo_mimic_joint_plugin.so" name="${name}_mimic_robotiq_85_1">
+		        <joint>${name}_right_driver_joint</joint>
+		        <mimicJoint>${name}_left_driver_joint</mimicJoint>
+		        <!--multiplier>1.0</multiplier>
+		        <offset>0.0</offset-->
+		    </plugin>
+		    <plugin filename="libroboticsgroup_gazebo_mimic_joint_plugin.so" name="${name}_mimic_robotiq_85_2">
+		        <joint>${name}_right_driver_joint</joint>
+		        <mimicJoint>${name}_left_follower_joint</mimicJoint>
+		        <!--multiplier>1.0</multiplier>
+		        <offset>0.0</offset-->
+		    </plugin>
+		    <plugin filename="libroboticsgroup_gazebo_mimic_joint_plugin.so" name="${name}_mimic_robotiq_85_3">
+		        <joint>${name}_right_driver_joint</joint>
+		        <mimicJoint>${name}_left_spring_link_joint</mimicJoint>
+		        <!--multiplier>1.0</multiplier>
+		        <offset>0.0</offset-->
+		    </plugin>
+		    <plugin filename="libroboticsgroup_gazebo_mimic_joint_plugin.so" name="${name}_mimic_robotiq_85_4">
+		        <joint>${name}_right_driver_joint</joint>
+		        <mimicJoint>${name}_right_follower_joint</mimicJoint>
+		        <multiplier>-1.0</multiplier>
+		        <offset>0.0</offset>
+		    </plugin>
+		    <plugin filename="libroboticsgroup_gazebo_mimic_joint_plugin.so" name="${name}_mimic_robotiq_85_5">
+		        <joint>${name}_right_driver_joint</joint>
+		        <mimicJoint>${name}_right_spring_link_joint</mimicJoint>
+		        <multiplier>-1.0</multiplier>
+		        <offset>0.0</offset>
+		    </plugin>
+		</gazebo>
 	</xacro:macro>
 </robot>
